File: esptopc_poweron_remote_pcb/esptopc_poweron_remote_pcb.kicad_pcb (KiCad board)
At the start: 2 copper layers, 38.6 x 22.4 mm, 23 parts, among them J1 Conn_01x05_Pin, Q1 IRLML6402, Q2 IRLML2502, Q3 IRLML6402, Q4 IRLML2502, Q5 IRLML2502, U1 AMS1117, U2 ESP-01

Commit message: Потерялась дорожка. Нашлась
Routing:
- net +3.3V: track 58.6 -> 62.5 mm
Changed lines of the file:
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@@
 		)
 		(fp_text user "${REFERENCE}"
-			(at 0 0 -90)
+			(at 0 0 270)
 			(layer "F.Fab")
 			(effects
@@
 	)
 	(segment
+		(start 171.2304 102.7532)
+		(end 172.212 103.7348)
+		(width 0.5)
+		(layer "F.Cu")
+		(net "LED+")
+	)
+	(segment
+		(start 169.5732 102.7532)
+		(end 170.9928 102.7532)
+		(width 0.5)
+		(layer "F.Cu")
+		(net "LED+")
+	)
+	(segment
+		(start 170.9928 102.7532)
+		(end 171.2304 102.7532)
+		(width 0.5)
+		(layer "F.Cu")
+		(net "LED+")
+	)
+	(via
+		(at 170.9928 102.7532)
+		(size 0.6)
+		(drill 0.3)
+		(layers "F.Cu" "B.Cu")
+		(net "LED+")
+	)
+	(segment
+		(start 172.466 97.79)
+		(end 172.466 99.1108)
+		(width 0.5)
+		(layer "B.Cu")
+		(net "LED+")
+	)
+	(segment
+		(start 170.9928 102.7532)
+		(end 170.9928 100.584)
+		(width 0.5)
+		(layer "B.Cu")
+		(net "LED+")
+	)
+	(segment
+		(start 172.466 99.1108)
+		(end 170.9928 100.584)
+		(width 0.5)
+		(layer "B.Cu")
+		(net "LED+")
+	)
+	(segment
+		(start 166.5732 101.8032)
+		(end 164.2326 101.8032)
+		(width 0.5)
+		(layer "F.Cu")
+		(net "Net-(Q5-D)")
+	)
+	(segment
+		(start 166.5732 100.9904)
+		(end 166.7256 100.838)
+		(width 0.5)
+		(layer "F.Cu")
+		(net "Net-(Q5-D)")
+	)
+	(segment
+		(start 166.5732 101.8032)
+		(end 166.5732 100.9904)
+		(width 0.5)
+		(layer "F.Cu")
+		(net "Net-(Q5-D)")
+	)
+	(segment
+		(start 164.2326 101.8032)
+		(end 164.131 101.9048)
+		(width 0.5)
+		(layer "F.Cu")
+		(net "Net-(Q5-D)")
+	)
+	(via
+		(at 166.7256 100.838)
+		(size 0.6)
+		(drill 0.3)
+		(layers "F.Cu" "B.Cu")
+		(net "Net-(Q5-D)")
+	)
+	(segment
+		(start 166.7256 100.838)
+		(end 167.412 100.838)
+		(width 0.5)
+		(layer "B.Cu")
+		(net "Net-(Q5-D)")
+	)
+	(segment
+		(start 167.412 100.838)
+		(end 169.698 98.552)
+		(width 0.5)
+		(layer "B.Cu")
+		(net "Net-(Q5-D)")
+	)
+	(segment
 		(start 159.004 104.394)
 		(end 161.4932 101.9048)
@@
 	)
 	(segment
+		(start 159.3596 93.5996)
+		(end 156.3364 93.5996)
+		(width 0.5)
+		(layer "F.Cu")
+		(net "+3.3V")
+	)
+	(segment
 		(start 161.798 92.7304)
 		(end 160.2288 92.7304)
@@
 	)
 	(segment
+		(start 156.3364 93.5996)
+		(end 155.702 94.234)
+		(width 0.5)
+		(layer "F.Cu")
+		(net "+3.3V")
+	)
+	(segment
 		(start 155.7405 91.694)
 		(end 158.47 91.694)
@@
 	)
 	(segment
-		(start 171.2304 102.7532)
-		(end 172.212 103.7348)
-		(width 0.5)
-		(layer "F.Cu")
-		(net "LED+")
-	)
-	(segment
-		(start 169.5732 102.7532)
-		(end 170.9928 102.7532)
-		(width 0.5)
-		(layer "F.Cu")
-		(net "LED+")
-	)
-	(segment
-		(start 170.9928 102.7532)
-		(end 171.2304 102.7532)
-		(width 0.5)
-		(layer "F.Cu")
-		(net "LED+")
-	)
-	(via
-		(at 170.9928 102.7532)
-		(size 0.6)
-		(drill 0.3)
-		(layers "F.Cu" "B.Cu")
-		(net "LED+")
-	)
-	(segment
-		(start 172.466 97.79)
-		(end 172.466 99.1108)
-		(width 0.5)
-		(layer "B.Cu")
-		(net "LED+")
-	)
-	(segment
-		(start 170.9928 102.7532)
-		(end 170.9928 100.584)
-		(width 0.5)
-		(layer "B.Cu")
-		(net "LED+")
-	)
-	(segment
-		(start 172.466 99.1108)
-		(end 170.9928 100.584)
-		(width 0.5)
-		(layer "B.Cu")
-		(net "LED+")
-	)
-	(segment
 		(start 170.2728 95.25)
 		(end 169.394 96.1288)
@@
 		(net "Net-(Q1-D)")
 	)
-	(segment
-		(start 166.5732 101.8032)
-		(end 164.2326 101.8032)
-		(width 0.5)
-		(layer "F.Cu")
-		(net "Net-(Q5-D)")
-	)
-	(segment
-		(start 166.5732 100.9904)
-		(end 166.7256 100.838)
-		(width 0.5)
-		(layer "F.Cu")
-		(net "Net-(Q5-D)")
-	)
-	(segment
-		(start 166.5732 101.8032)
-		(end 166.5732 100.9904)
-		(width 0.5)
-		(layer "F.Cu")
-		(net "Net-(Q5-D)")
-	)
-	(segment
-		(start 164.2326 101.8032)
-		(end 164.131 101.9048)
-		(width 0.5)
-		(layer "F.Cu")
-		(net "Net-(Q5-D)")
-	)
-	(via
-		(at 166.7256 100.838)
-		(size 0.6)
-		(drill 0.3)
-		(layers "F.Cu" "B.Cu")
-		(net "Net-(Q5-D)")
-	)
-	(segment
-		(start 166.7256 100.838)
-		(end 167.412 100.838)
-		(width 0.5)
-		(layer "B.Cu")
-		(net "Net-(Q5-D)")
-	)
-	(segment
-		(start 167.412 100.838)
-		(end 169.698 98.552)
-		(width 0.5)
-		(layer "B.Cu")
-		(net "Net-(Q5-D)")
-	)
 	(zone
